Commit message: Added bot model to launch file

File: fsm_bot_description/urdf/fsm_bot.xacro (robot description, xacro)
@@ -138,5 +138,5 @@
   <parent link="motor_right_1"/>
   <child link="tyre_right_1"/>
-  <axis xyz="1.0 0.0 -0.0"/>
+  <axis xyz="-1.0 0.0 -0.0"/>
 </joint>
 <joint name="Revolute 7" type="continuous">
